File: Projects/I2C Expansion Card/USBC_I2C Kicad/USBC_I2C.kicad_sch (KiCad schematic)
At the start: 12 parts, among them P1 USB_C_Plug_USB2.0, U2 MCP2221AxP

Commit message: Worked on KiCad Schematic
Parts:
- removed C1, C3: C_Small, symbol Device:C_Small
- removed D1, D2, D3, D5: LED, symbol Device:LED
- removed R1, R2, R3, R4: R, symbol Device:R
- added C1, C2: C, symbol Device:C
- added D1: 1206 SMD LEDS, LED_SMD:LED_1206_3216Metric, symbol LED:IR26-21C_L110_TR8
- added D2, D3, D4: IR26-21C_L110_TR8, LED_SMD:LED_1206_3216Metric, symbol LED:IR26-21C_L110_TR8
- added R1: Resistors TBD, symbol Device:R_US
- added R2, R3, R4: R_US, symbol Device:R_US
- U1: renamed from U2; value MCP2221AxP -> MCP2221A
- USB1: renamed from P1; value USB_C_Plug_USB2.0 -> USB C Male Connector
Connections:
- net GND: now also USB1.S1 (SHIELD), C1.1, C2.1, R1.2, R2.2, R3.2, R4.2
- net at U1.7 (GP2): now also D3.2 (A)
- net 5V: now reaches U1.1 (VDD), USB1.A4 (VBUS), USB1.A9 (VBUS), USB1.B4 (VBUS), USB1.B9 (VBUS)
- net 5V: now also C1.2
- net at U1.11 (VUSB): now also C2.2
- net at U1.2 (GP0): now also D1.2 (A)
- net at U1.8 (GP3): now also D4.2 (A)
- net at U1.3 (GP1): now also D2.2 (A)
- net SCL: now reaches U1.10 (SCL)
- net SDA: now reaches U1.9 (SDA)
- new net: D2.1 (K), R2.1
- new net: D3.1 (K), R3.1
- new net: D4.1 (K), R4.1
- new net: D1.1 (K), R1.1
Other:
- note added: "**Use Nonpolarized Caps Rev 1 - Seth Gaboury: Created basic Digital Keycad schematic for the USBC to I2C, Need to double check connections as this was a rough draft and kinda tough on track pad Rev 1.1 - Bradley Burkard: Updated it with potential choice of SMD LEDs, and rerouted some connections for ease of viewing. Added location for I2C Out"
- note added: "I2C Output"
- note added: "Indicator LEDs"
- note added: "UART Interface (Not priority)"
- note added: "URx UTx USB Status I2C"
- note added: "USB > I2C Interface"
- note removed: "**Use Unpolarized Capacitors"
- note removed: "R"
- note removed: "Rev 1 - Seth Gaboury: Created basic Digital Keycad schematic for the USBC to I2C, Need to double check connections as this was a rough draft and kinda tough on track pad,"

Commit message: Updated USB to I2C
added values and updated schematic
Parts:
- added R5: 10K, symbol Device:R_US
- C1: value C -> 1 μF
- C2: value C -> 0.47 μF
- R1: value Resistors TBD -> Resistors 1K Ohm
Connections:
- net 5V: now also R5.2
- net GND: now also C2.2; no longer C2.1
- net at U1.11 (VUSB): now also C2.1; no longer C2.2
- net at U1.4 (~{RST}): now also R5.1
Other:
- note added: "** C1 MUST NOT BE BELOW 10 μF OR INRUSH CURRENT PROTECTION IS REQUIRED"
- note added: "4 Pin Header"
- note added: "Rev 1.2 - Seth Gaboury: Updated schematic and implemented values for many of the components, please review the changes"
- moved on the sheet: C2
